File: Sweep half-swept/half-swept.kicad_pcb (KiCad board)
At the start: 2 copper layers, 109 x 86.9 mm, 25 parts, among them J2 AudioJack4dpb, SW1 SW_Push, SW10 SW_Push, SW11 SW_Push, SW12 SW_Push, SW13 SW_Push, SW14 SW_Push, SW15 SW_Push, SW16 SW_Push, SW17 SW_Push, SW2 SW_Push, SW3 SW_Push, SW4 SW_Push, SW5 SW_Push, SW6 SW_Push, SW7 SW_Push, SW8 SW_Push, SW9 SW_Push, U1 ProMicro-kbd

Commit message: experimental mods
Parts:
- removed the G*** at (64.0, 82.0)
- removed J2: AudioJack4dpb, Kailh:TRRS-PJ-DPB2
- removed POWER SW: SW_SPDT, Kailh:SPDT_C128955
- removed REF**: Tenting Puck, kbd:Tenting_Puck2
- added G***: LOGO, Custom Footprints:ferris, F.Cu at (65.8, 83.0)
- added RSW4: SW_Push, * duckyb-collection:Tactile-Switch_SMT, F.Cu at (122.0, 81.4)
- added SW_POWER1: SK12D07VG4, SK12D07VG4:SK12D07VG4, F.Cu at (45.5, 81.3)
- moved RSW2 66.7 mm to (115.7, 81.4)
- moved B+ 1.89 mm to (124.6, 46.0)
- moved B- 1.26 mm to (112.5, 45.8)
- moved U1 0.40 mm to (118.5, 63.0)
- renumbered SW8 to SW10, SW9 to SW11, SW10 to SW12, SW11 to SW14, SW12 to SW15, SW13 to SW16, SW14 to SW17, SW15 to SW18, SW1 to SW2, SW17 to SW20, SW16 to SW21, SW2 to SW3, SW3 to SW4, SW4 to SW5, SW5 to SW6, SW6 to SW8, SW7 to SW9
Connections:
- B+ pad 1: BT+_r -> BT+
- RSW2 pad 1: gnd -> reset
- RSW2 pad 2: gnd -> reset
- SW20 pad 1: Switch17 -> Switch16
- SW21 pad 1: Switch16 -> Switch17
- U1 pad 10: Switch1 -> Switch15
- U1 pad 9: Switch15 -> Switch1
Routing:
- net BT+: track 0.00 -> 103.7 mm, vias 0 -> 2
- net raw: track 42.9 -> 98.4 mm
- net BT+_r: track 50.6 -> 0.00 mm, vias 2 -> 0
- net vcc: track 48.8 -> 0.00 mm, vias 4 -> 0
- net gnd: track 15.1 -> 27.2 mm, vias 3 -> 2
- net Switch17: track 21.5 -> 27.2 mm
- net Net-(SW_POWERR1-Pad1): track 5.39 -> 0.00 mm, vias 1 -> 0
- net Switch16: track 24.6 -> 19.4 mm
- net Switch10: track 19.2 -> 23.4 mm
- net reset: track 49.7 -> 46.3 mm, vias 1 -> 6
- net Switch2: track 94.9 -> 92.1 mm
- net Switch11: track 107.5 -> 105.2 mm
- net Switch3: track 73.0 -> 70.8 mm
- net Switch18: track 34.4 -> 32.8 mm, vias 0 -> 1
- net Switch13: track 58.5 -> 60.0 mm
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Other:
- board text added: "0 1"
- board text added: "1 0"
- board text added: "Lean Half Swept"
- board text added: "SW_POWER1"
- board text removed: "Half Swept"
- board text removed: "TRRS"
